File: KiCad/SF500.sch (KiCad schematic (older format))
At the start: 37 parts, among them J1 Conn_01x06, J2 Conn_01x05, U1 68000D_MB_socket, U2 68000D_CPU_socket, U3 LM1117-3.3, U4 NB3N502, U5 CY62167G-48TSOP-I, U6 CY62167G-48TSOP-I, U7 CY62167G-48TSOP-I, U8 CY62167G-48TSOP-I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

Commit message: fixed modified symbol 68000D to reside in SF500.lib
Parts:
- U1: footprint Package_DIP:DIP-64_W22.86mm_LongPads -> SF500:DIP-64_W22.86mm_LongPads
- U2: symbol CPU_NXP_68000:68000D -> SF500:68000D
Changed lines of the file:
@@
 BG
 $Comp
-L CPU_NXP_68000:68000D U2
+L SF500:68000D U2
 U 1 1 5F7C541F
 P 4500 2950
@@
 F 0 "U1" H 1900 2850 50  0000 C CNN
 F 1 "68000D_MB_socket" H 1900 2950 50  0000 C CNN
-F 2 "Package_DIP:DIP-64_W22.86mm_LongPads" H 1900 2950 50  0001 C CNN
+F 2 "SF500:DIP-64_W22.86mm_LongPads" H 1900 2950 50  0001 C CNN
 F 3 "https://www.nxp.com/docs/en/reference-manual/MC68000UM.pdf" H 1900 2950 50  0001 C CNN
 	1    1900 2950
